Commit message: Task 2 added

File: eyrc-2022_holabot/urdf/hola_bot.urdf (robot description, URDF)
Before this commit: robot hola_bot, 4 links, 3 joints
Links:
- link base_link: mass 0.49 -> 1; geometry collision cylinder length=0.005 radius=0.15; visual mesh filename=package://eyrc-2022_holabot/meshes/base_link.obj
- link front_wheel: mass 0.062 -> 0.060
- link left_wheel: mass 0.062 -> 0.060
- link right_wheel: mass 0.062 -> 0.060
Joints:
- joint front_joint: origin xyz=0 0.17483 -0.0335 rpy=0 0 0 -> xyz=0 0.17483 0 rpy=0 0 0; type continuous -> revolute
- joint left_joint: axis 0 -1 0 -> 0 1 0; origin xyz=-0.15154 -0.087275 -0.0335 rpy=0 0 -1.04688 -> xyz=-0.15154 -0.087275 0 rpy=0 0 2.094; type continuous -> revolute
- joint right_joint: axis 0 -1 0 -> 0 1 0; origin xyz=0.15154 -0.087275 -0.0335 rpy=0 0 1.04688 -> xyz=0.15154 -0.087275 0 rpy=0 0 -2.094; type continuous -> revolute
